File: arrowhead.kicad_pcb (KiCad board)
At the start: 2 copper layers, 293.6 x 165.7 mm, 145 parts, among them J1 USB_C_Receptacle_USB2.0_14P, J2 USB_C_Receptacle_USB2.0_14P, J3 USB3_A, J4 USB3_A, U1 CH334R, Y1 Crystal_GND23

Commit message: realised the ch334 models aren't available from dk, so I had to redesign
Parts:
- added R3: Resistor, ScottoKeebs_Components:Resistor_0402, F.Cu at (201.5, 68.5)
- added R4: Resistor, ScottoKeebs_Components:Resistor_0402, F.Cu at (201.0, 187.0)
- U1: value CH334R -> TUSB2046BVF; footprint Package_SO:QSOP-16_3.9x4.9mm_P0.635mm -> footprints:VF32
- moved Y1 19.1 mm to (212.5, 123.4), turned to 0 degrees
- moved D15 13.0 mm to (131.7, 74.7), turned to 75 degrees
- moved D30 13.0 mm to (181.1, 110.3), turned to 75 degrees
- moved D5 13.0 mm to (173.3, 66.1), turned to 75 degrees
- moved D29 13.0 mm to (163.4, 102.9), turned to 75 degrees
- moved D4 13.0 mm to (155.6, 58.8), turned to 75 degrees
- moved D40 13.0 mm to (140.8, 114.0), turned to 75 degrees
- moved D53 13.0 mm to (153.6, 139.7), turned to 75 degrees
- moved D54 13.0 mm to (171.3, 147.1), turned to 75 degrees
- moved D25 13.0 mm to (88.8, 88.0), turned to 75 degrees
- moved D27 13.0 mm to (126.7, 93.1), turned to 75 degrees
- moved D37 13.0 mm to (83.8, 106.4), turned to 75 degrees
- moved D38 13.0 mm to (102.3, 111.3), turned to 75 degrees
- moved D2 13.0 mm to (117.0, 56.1), turned to 75 degrees
- moved D3 13.0 mm to (136.6, 56.3), turned to 75 degrees
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Connections:
- J1 pad A6: Net-(U1-DPU+) -> Net-(U1-DP0)
- J1 pad A7: Net-(U1-DMU-) -> Net-(U1-DM0)
- J1 pad B5: Net-(J1-CC1) -> Net-(J1-CC2)
- J1 pad B6: Net-(U1-DPU+) -> Net-(U1-DP0)
- J1 pad B7: Net-(U1-DMU-) -> Net-(U1-DM0)
- J2 pad A6: Net-(U1-DP4+) -> Net-(U1-DP1)
- J2 pad A7: Net-(U1-DM4-) -> Net-(U1-DM1)
- J2 pad B5: Net-(J2-CC1) -> Net-(J2-CC2)
- J2 pad B6: Net-(U1-DP4+) -> Net-(U1-DP1)
- J2 pad B7: Net-(U1-DM4-) -> Net-(U1-DM1)
- R2 pad 2: Net-(J2-CC1) -> Net-(J2-CC2)
- U1 pad 1: Net-(U1-DM4-) -> Net-(U1-DP0)
- U1 pad 10: Net-(U1-DMU-) -> VCC
- U1 pad 11: Net-(U1-DPU+) -> Net-(U1-DM1)
- U1 pad 12: unconnected-(U1-V5-Pad12) -> Net-(U1-DP1)
- U1 pad 14: GND -> VCC
- U1 pad 15: Net-(U1-XO) -> Net-(J4-D-)
- U1 pad 16: Net-(U1-XI) -> Net-(J4-D+)
- U1 pad 2: Net-(U1-DP4+) -> Net-(U1-DM0)
- U1 pad 3: Net-(J4-D-) -> VCC
- U1 pad 4: Net-(J4-D+) -> unconnected-(U1-*RESET-Pad4)
- U1 pad 5: Net-(J3-D-) -> unconnected-(U1-EECLK-Pad5)
- U1 pad 6: Net-(J3-D+) -> unconnected-(U1-EEDATA/GANGED-Pad6)
- U1 pad 7: Net-(U1-DM1-) -> GND
- U1 pad 8: Net-(U1-DP1+) -> GND
- U2 pad 1: Net-(U1-DP1+) -> Net-(U1-DP4)
- U2 pad 14: Net-(U1-DM1-) -> Net-(U1-DM4)
- Y1 pad 1: Net-(U1-XO) -> Net-(U1-XTAL1)
- Y1 pad 4: Net-(U1-XI) -> Net-(U1-XTAL2)
Routing:
- net ROW4: track 348.5 -> 0.00 mm, vias 13 -> 0
- net ROW3: track 316.1 -> 0.00 mm, vias 12 -> 0
- net ROW0: track 285.3 -> 0.00 mm, vias 13 -> 0
- net ROW2: track 274.0 -> 0.00 mm, vias 13 -> 0
- net ROW1: track 266.7 -> 0.00 mm, vias 12 -> 0
- net COL1: track 82.2 -> 0.00 mm, vias 5 -> 0
- net COL9: track 81.8 -> 0.00 mm, vias 5 -> 0
- net COL8: track 81.8 -> 0.00 mm, vias 5 -> 0
- net COL5: track 81.8 -> 0.00 mm, vias 5 -> 0
- net COL2: track 81.8 -> 0.00 mm, vias 5 -> 0
- net COL10: track 81.8 -> 0.00 mm, vias 5 -> 0
- net COL4: track 81.8 -> 0.00 mm, vias 5 -> 0
- net COL3: track 81.8 -> 0.00 mm, vias 5 -> 0
- net COL11: track 81.8 -> 0.00 mm, vias 5 -> 0
- net COL0: track 81.8 -> 0.00 mm, vias 5 -> 0
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- added copper zone on B.Cu, net GND
- added copper zone on F.Cu, net vbus
Other:
- board text added: "Arrowhead"
- board text added: "Don't Panic"
- board text added: "It was walpole"
- board text added: "M1racleMax"
- board text added: "Peace and long life"
- board text added: "Roll for initiative"
- board text added: "WayWayWay"

Commit message: production run 1
Parts:
- added C1: C_US, Capacitor_SMD:C_0603_1608Metric_Pad1.08x0.95mm_HandSolder, F.Cu at (209.9, 125.6)
- added C2: C_US, Capacitor_SMD:C_0603_1608Metric_Pad1.08x0.95mm_HandSolder, F.Cu at (212.7, 122.1)
- added D69: LED, LED_SMD:LED_0603_1608Metric_Pad1.05x0.95mm_HandSolder, F.Cu at (211.8, 119.6)
- Y1: footprint Crystal:Crystal_SMD_2520-4Pin_2.5x2.0mm -> Crystal:Crystal_SMD_7050-4Pin_7.0x5.0mm
- moved Y1 5.93 mm to (218.4, 124.3)
- moved R3 4.11 mm to (201.5, 72.6)
- moved R2 2.31 mm to (205.0, 190.2)
- moved R1 1.99 mm to (206.5, 68.8)
- turned U1 to -90 degrees
Connections:
- J2 pad A6: Net-(U1-DP1) -> Net-(U1-DP3)
- J2 pad A7: Net-(U1-DM1) -> Net-(U1-DM3)
- J2 pad B6: Net-(U1-DP1) -> Net-(U1-DP3)
- J2 pad B7: Net-(U1-DM1) -> Net-(U1-DM3)
- U1 pad 11: Net-(U1-DM1) -> Net-(J3-D-)
- U1 pad 12: Net-(U1-DP1) -> Net-(J3-D+)
- U1 pad 19: Net-(J3-D-) -> Net-(U1-DM3)
- U1 pad 20: Net-(J3-D+) -> Net-(U1-DP3)
- U1 pad 26: unconnected-(U1-*EXTMEM-Pad26) -> VCC
- U1 pad 27: unconnected-(U1-TSTPLL/48MCLK-Pad27) -> GND
- U1 pad 31: unconnected-(U1-TSTMODE-Pad31) -> GND
- U1 pad 32: unconnected-(U1-SUSPND-Pad32) -> Net-(D69-A)
- U1 pad 4: unconnected-(U1-*RESET-Pad4) -> VCC
- U1 pad 6: unconnected-(U1-EEDATA/GANGED-Pad6) -> VCC
- Y1 pad 1: Net-(U1-XTAL1) -> Net-(U1-XTAL2)
- Y1 pad 4: Net-(U1-XTAL2) -> Net-(U1-XTAL1)
Routing:
- net ROW4: track 0.00 -> 345.8 mm, vias 0 -> 2
- net ROW3: track 0.00 -> 324.4 mm, vias 0 -> 2
- net ROW2: track 0.00 -> 317.3 mm, vias 0 -> 2
- net ROW1: track 0.00 -> 266.1 mm
- net COL2: track 0.00 -> 258.6 mm
- net ROW0: track 0.00 -> 254.3 mm
- net ROW5: track 0.00 -> 252.1 mm, vias 0 -> 2
- net COL3: track 0.00 -> 240.4 mm
- net GND: track 0.00 -> 235.4 mm, vias 0 -> 38
- net COL0: track 0.00 -> 226.8 mm
- net COL4: track 0.00 -> 223.7 mm
- net COL11: track 0.00 -> 222.5 mm, vias 0 -> 2
- net COL9: track 0.00 -> 221.7 mm, vias 0 -> 1
- net COL1: track 0.00 -> 208.8 mm
- net COL8: track 0.00 -> 203.8 mm, vias 0 -> 1
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Other:
- board text removed: "It was walpole"
- board text removed: "Peace and long life"
- board text removed: "Roll for initiative"

Commit message: actual first production run
Routing:
- net GND: track 235.4 -> 256.4 mm, vias 38 -> 36
- net ROW5: track 252.1 -> 245.1 mm, vias 2 -> 0
- net vbus: track 26.5 -> 33.2 mm
- net Net-(D68-A): track 4.70 -> 7.24 mm
- net COL10: track 198.5 -> 196.9 mm
- net Net-(U1-DM0): track 60.5 -> 58.9 mm
- net Net-(D57-A): track 4.54 -> 5.72 mm
- net Net-(D45-A): track 4.54 -> 5.53 mm
- net Net-(D44-A): track 4.54 -> 5.44 mm
- net Net-(D63-A): track 4.54 -> 5.40 mm
- net COL11: track 222.5 -> 221.6 mm
- net Net-(D11-A): track 4.54 -> 5.37 mm
- net Net-(D65-A): track 4.54 -> 5.36 mm
- net Net-(D47-A): track 4.54 -> 5.34 mm
- net Net-(D36-A): track 4.54 -> 5.34 mm
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